Commit message: init

File: chapt6/chapt6_ws/src/fishbot_description/urdf/fishbot/fishbot.urdf.xacro (robot description, xacro)
@@ -16,7 +16,9 @@
 <xacro:include filename="$(find fishbot_description)/urdf/fishbot/actuator/caster.urdf.xacro"/>   <!--$(find fishbot_description)表示找到share目录下的fishbot_description(功能包的名字)目录-->
 <!-- 插件 控制机器人运动插件-->
-<xacro:include filename="$(find fishbot_description)/urdf/fishbot/plugins/gazebo_control_plugin.xacro"/>   <!--$(find fishbot_description)表示找到share目录下的fishbot_description(功能包的名字)目录-->
+<xacro:include filename="$(find fishbot_description)/urdf/fishbot/plugins/gazebo_control_plugin.xacro"/>   $(find fishbot_description)表示找到share目录下的fishbot_description(功能包的名字)目录
 <!-- 插件 机器人的传感器插件-->
 <xacro:include filename="$(find fishbot_description)/urdf/fishbot/plugins/gazebo_sensor_plugin.xacro"/>   <!--$(find fishbot_description)表示找到share目录下的fishbot_description(功能包的名字)目录-->
+<!-- 插件 使用ros2_control来控制机器人运动；其与gazebo中的两轮差速插件运动控制会有冲突，所以同时只能使用一个插件来控制机器人运动 -->
+<xacro:include filename="$(find fishbot_description)/urdf/fishbot/fishbot.ros2_control.xacro"/>   <!--$(find fishbot_description)表示找到share目录下的fishbot_description(功能包的名字)目录-->
 <!-- 调用宏 -->
 <xacro:base_xacro length="0.12" radius="0.10"/>
@@ -30,5 +32,6 @@
 <xacro:caster_xacro caster_name="back_caster" xyz="-0.08 0.0 -0.076"/> <!--   -0.08 表示沿着X轴反方向偏移0.08 -0.076表示沿着Z轴向下偏移0.076-->
 <!-- 使用插件 -->
-<xacro:gazebo_control_plugin />
+<!-- <xacro:gazebo_control_plugin /> -->
 <xacro:gazebo_sensor_plugin />
+<xacro:fishbot_ros2_control />
 </robot>

File: chapt6/chapt6_ws/src/fishbot_description/urdf/fishbot/plugins/gazebo_sensor_plugin.xacro (robot description, xacro)
@@ -115,3 +115,31 @@
     </gazebo>
     </xacro:macro>
+    <gazebo reference="camera_link">
+        <!-- gazebo的插件，这个插件用于给camera_link(传感器部件名称)添加深度相机传感器仿真 -->
+        <sensor type="depth" name="camera_sensor">
+            <plugin name="depth_camera" filename="libgazebo_ros_camera.so">
+                <!-- 传感器数据会供应到camera_optical_link上 -->
+                <frame_name>camera_optical_link</frame_name>
+            </plugin>
+            <always_on>true</always_on>
+            <update_rate>10</update_rate>
+            <camera name="camera">
+                <horizontal_fov>1.5009831567</horizontal_fov>  <!--90度-->
+                <image>
+                    <width>800</width>
+                    <height>600</height>
+                    <format>R8G8B8</format>
+                </image>
+                <!-- 机变系数，仿真相机无所谓 -->
+                <distortion>
+                    <k1>0.0</k1>
+                    <k2>0.0</k2>
+                    <k3>0.0</k3>
+                    <p1>0.0</p1>
+                    <p2>0.0</p2>
+                    <center>0.5 0.5</center>
+                </distortion>
+            </camera>
+        </sensor>
+    </gazebo>
 </robot>

File: chapt6/chapt6_ws/src/fishbot_description/urdf/fishbot/sensor/camera.urdf.xacro (robot description, xacro)
@@ -39,4 +39,6 @@
             <xacro:box_inertia m="0.1" w="0.02" h="0.10" d="0.02" />
         </link>
+        <!-- 创建虚拟部件 -->
+        <link name="camera_optical_link"></link>
         <!-- 机器人的关节，用于组合机器人的部件，此处将camera_link和base_link进行组合 -->
         <joint name="camera_jonit" type="fixed">  <!--fixed表示固定死的-->
@@ -47,4 +49,12 @@
             <origin xyz="${xyz}" rpy="0.0 0.0 0.0"/>
         </joint>
+        <!-- 虚拟部件的关节 -->
+        <joint name="camera_optical_jonit" type="fixed">  <!--fixed表示固定死的-->
+            <!-- 目前的意思表示将camera_optical_link固定在camera_link上面 -->
+            <parent link="camera_link"/> <!--父部件-->
+            <child link="camera_optical_link"/> <!--子部件-->
+            <!-- 固定的位置，偏移和旋转 -->
+            <origin xyz="0 0 0" rpy="${-pi/2} 0.0 ${-pi/2}"/>
+        </joint>
     </xacro:macro>
 </robot>
